File: cp2102_header.kicad_pcb (KiCad board)
At the start: 2 copper layers, 13.3 x 22.9 mm, 24 parts, among them J1 FTDI, J2 USB_B_Micro, J8 Serial, Q3 BSS138PS, U2 CP2102N

Commit message: move around / tidy-up labels
Other:
- board text added: "200131"
- board text removed: "200122"
Changed lines of the file:
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@@
       (effects (font (size 1 1) (thickness 0.15)))
     )
-    (fp_text value 330 (at 0 0 180) (layer F.SilkS)
+    (fp_text value 330 (at 0 -0.127 180) (layer F.SilkS)
       (effects (font (size 0.6 0.6) (thickness 0.125)))
     )
@@
     )
   )
-  (gr_text 200122 (at 84.836 86.36 90) (layer B.SilkS)
+  (gr_text 200131 (at 84.836 86.36 90) (layer B.SilkS)
     (effects (font (size 0.7 0.7) (thickness 0.15)) (justify mirror))
   )
-  (gr_text GND. (at 81.407 72.060952) (layer F.SilkS)
+  (gr_text GND. (at 81.407 72.187952) (layer F.SilkS)
     (effects (font (size 0.7 0.7) (thickness 0.15)))
   )
-  (gr_text GND. (at 81.0895 72.0725) (layer B.SilkS)
+  (gr_text GND. (at 81.0895 72.1995) (layer B.SilkS)
     (effects (font (size 0.7 0.7) (thickness 0.15)) (justify mirror))
   )
-  (gr_text RXD. (at 86.487 72.009) (layer F.SilkS)
+  (gr_text RXD. (at 86.487 72.136) (layer F.SilkS)
     (effects (font (size 0.7 0.7) (thickness 0.15)))
   )
-  (gr_text RXD. (at 86.233 72.009) (layer B.SilkS)
+  (gr_text RXD. (at 86.233 72.136) (layer B.SilkS)
     (effects (font (size 0.7 0.7) (thickness 0.15)) (justify mirror))
   )
-  (gr_text TXD. (at 84.074 72.009) (layer F.SilkS)
+  (gr_text TXD. (at 84.074 72.136) (layer F.SilkS)
     (effects (font (size 0.7 0.7) (thickness 0.15)))
   )
-  (gr_text TXD. (at 83.566 72.009) (layer B.SilkS)
+  (gr_text TXD. (at 83.566 72.136) (layer B.SilkS)
     (effects (font (size 0.7 0.7) (thickness 0.15)) (justify mirror))
   )
-  (gr_text GND. (at 89.027 72.009) (layer F.SilkS)
+  (gr_text GND. (at 89.027 72.136) (layer F.SilkS)
     (effects (font (size 0.7 0.7) (thickness 0.15)))
   )
-  (gr_text GND. (at 88.773 72.009) (layer B.SilkS)
+  (gr_text GND. (at 88.773 72.136) (layer B.SilkS)
     (effects (font (size 0.7 0.7) (thickness 0.15)) (justify mirror))
   )
-  (gr_text VIO (at 88.646 93.472) (layer F.SilkS)
-    (effects (font (size 0.6 0.6) (thickness 0.125)))
+  (gr_text VIO (at 88.646 93.345) (layer F.SilkS)
+    (effects (font (size 0.4 0.6) (thickness 0.1)))
   )
-  (gr_text VIO (at 88.646 93.472) (layer B.SilkS)
-    (effects (font (size 0.6 0.6) (thickness 0.125)) (justify mirror))
+  (gr_text VIO (at 88.646 93.345) (layer B.SilkS)
+    (effects (font (size 0.4 0.6) (thickness 0.1)) (justify mirror))
   )
   (gr_line (start 89.154 83.82) (end 89.408 83.82) (layer B.SilkS) (width 0.2))
@@
   (gr_line (start 87.122 78.74) (end 89.154 78.74) (layer F.SilkS) (width 0.2))
   (gr_line (start 87.122 76.2) (end 89.154 76.2) (layer F.SilkS) (width 0.2))
-  (gr_text 200122 (at 84.836 86.36 90) (layer F.SilkS)
+  (gr_text 200131 (at 84.836 86.36 90) (layer F.SilkS)
     (effects (font (size 0.7 0.7) (thickness 0.15)))
   )
@@
     (effects (font (size 0.7 0.7) (thickness 0.15)) (justify mirror))
   )
-  (gr_text 5V (at 90.678 91.186) (layer B.SilkS)
+  (gr_text 5V (at 90.424 91.059) (layer B.SilkS)
     (effects (font (size 0.6 0.6) (thickness 0.125)) (justify mirror))
   )
-  (gr_text 3.3V (at 86.233 91.186) (layer B.SilkS)
+  (gr_text 3.3V (at 86.36 91.059) (layer B.SilkS)
     (effects (font (size 0.6 0.6) (thickness 0.125)) (justify mirror))
   )
@@
     (effects (font (size 0.7 0.7) (thickness 0.15)))
   )
-  (gr_text 3.3V (at 86.36 91.186) (layer F.SilkS)
+  (gr_text 3.3V (at 86.487 91.059) (layer F.SilkS)
     (effects (font (size 0.5 0.5) (thickness 0.125)))
   )
-  (gr_text 5V (at 90.678 91.186) (layer F.SilkS)
+  (gr_text 5V (at 90.424 91.059) (layer F.SilkS)
     (effects (font (size 0.6 0.6) (thickness 0.125)))
   )

Commit message: revert back to previous version
Other:
- board text added: "201224"
- board text removed: "200131"
Changed lines of the file:
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@@
     )
   )
-  (gr_text 200131 (at 84.836 86.36 90) (layer B.SilkS)
+  (gr_text 201224 (at 84.836 86.36 90) (layer B.SilkS)
     (effects (font (size 0.7 0.7) (thickness 0.15)) (justify mirror))
   )
@@
   (gr_line (start 87.122 78.74) (end 89.154 78.74) (layer F.SilkS) (width 0.2))
   (gr_line (start 87.122 76.2) (end 89.154 76.2) (layer F.SilkS) (width 0.2))
-  (gr_text 200131 (at 84.836 86.36 90) (layer F.SilkS)
+  (gr_text 201224 (at 84.836 86.36 90) (layer F.SilkS)
     (effects (font (size 0.7 0.7) (thickness 0.15)))
   )
